Commit message: URDF xacro: mesh-derived link inertials
Replace placeholder round-number masses/inertias with mesh-derived values
(compute_inertia.py) for all six arm links + suction_cup. cuRobo ignores
these, but they make the xacro consistent with the live URDF.

Co-Authored-By: Claude Opus 4.8 <noreply@anthropic.com>

File: src/mycobot_description/urdf/mycobot_pro_630.urdf.xacro (robot description, xacro)
@@ -38,7 +38,7 @@
     </collision>
     <inertial>
-      <mass value="1.0"/>
-      <origin xyz="0 0 0.1" rpy="0 0 0"/>
-      <inertia ixx="0.01" ixy="0" ixz="0" iyy="0.01" iyz="0" izz="0.01"/>
+      <mass value="3.4225"/>
+      <origin xyz="-0.01340 0.00001 0.06584" rpy="0 0 0"/>
+      <inertia ixx="1.129165e-02" ixy="5.520573e-08" ixz="-1.427358e-04" iyy="1.123173e-02" iyz="-2.051531e-07" izz="9.902095e-03"/>
     </inertial>
   </link>
@@ -58,7 +58,7 @@
     </collision>
     <inertial>
-      <mass value="0.5"/>
-      <origin xyz="0 0 -0.03" rpy="0 0 0"/>
-      <inertia ixx="0.005" ixy="0" ixz="0" iyy="0.005" iyz="0" izz="0.005"/>
+      <mass value="0.5434"/>
+      <origin xyz="0.00000 0.00756 -0.01455" rpy="0 0 0"/>
+      <inertia ixx="5.668835e-04" ixy="-3.760352e-12" ixz="9.896184e-13" iyy="5.117732e-04" iyz="-4.413917e-05" izz="4.049449e-04"/>
     </inertial>
   </link>
@@ -86,7 +86,7 @@
     </collision>
     <inertial>
-      <mass value="0.4"/>
-      <origin xyz="0.135 0 0" rpy="0 0 0"/>
-      <inertia ixx="0.004" ixy="0" ixz="0" iyy="0.004" iyz="0" izz="0.004"/>
+      <mass value="1.8125"/>
+      <origin xyz="0.13444 0.00002 -0.07533" rpy="0 0 0"/>
+      <inertia ixx="1.228935e-03" ixy="-1.272130e-06" ixz="-2.471483e-08" iyy="1.586526e-02" iyz="-9.612172e-09" izz="1.590244e-02"/>
     </inertial>
   </link>
@@ -114,7 +114,7 @@
     </collision>
     <inertial>
-      <mass value="0.3"/>
-      <origin xyz="0.1335 0 0" rpy="0 0 0"/>
-      <inertia ixx="0.003" ixy="0" ixz="0" iyy="0.003" iyz="0" izz="0.003"/>
+      <mass value="2.2651"/>
+      <origin xyz="0.12248 -0.00023 0.00100" rpy="0 0 0"/>
+      <inertia ixx="2.064878e-03" ixy="-1.732790e-06" ixz="-3.721500e-04" iyy="1.966886e-02" iyz="-9.829410e-08" izz="1.904045e-02"/>
     </inertial>
   </link>
@@ -142,7 +142,7 @@
     </collision>
     <inertial>
-      <mass value="0.2"/>
-      <origin xyz="0 -0.0475 0" rpy="0 0 0"/>
-      <inertia ixx="0.002" ixy="0" ixz="0" iyy="0.002" iyz="0" izz="0.002"/>
+      <mass value="0.3447"/>
+      <origin xyz="-0.00000 -0.01491 0.00910" rpy="0 0 0"/>
+      <inertia ixx="2.681047e-04" ixy="-2.278568e-08" ixz="4.082182e-09" iyy="1.881600e-04" iyz="-2.695459e-05" izz="2.437713e-04"/>
     </inertial>
   </link>
@@ -170,7 +170,7 @@
     </collision>
     <inertial>
-      <mass value="0.15"/>
-      <origin xyz="-0.027 0 0" rpy="0 0 0"/>
-      <inertia ixx="0.001" ixy="0" ixz="0" iyy="0.001" iyz="0" izz="0.001"/>
+      <mass value="0.4204"/>
+      <origin xyz="0.00078 -0.00000 -0.00654" rpy="0 0 0"/>
+      <inertia ixx="2.502357e-04" ixy="1.986448e-12" ixz="-2.156206e-06" iyy="3.887104e-04" iyz="-3.526369e-12" izz="3.525862e-04"/>
     </inertial>
   </link>
@@ -198,7 +198,7 @@
     </collision>
     <inertial>
-      <mass value="0.1"/>
-      <origin xyz="0.01 0 0" rpy="0 0 0"/>
-      <inertia ixx="0.0005" ixy="0" ixz="0" iyy="0.0005" iyz="0" izz="0.0005"/>
+      <mass value="0.0376"/>
+      <origin xyz="0.00543 0.00000 -0.00000" rpy="0 0 0"/>
+      <inertia ixx="1.679697e-05" ixy="-1.012847e-13" ixz="8.043638e-10" iyy="8.708365e-06" iyz="6.140298e-13" izz="8.708534e-06"/>
     </inertial>
   </link>
@@ -227,7 +227,7 @@
     </collision>
     <inertial>
-      <mass value="0.05"/>
-      <origin xyz="0 0 0.025" rpy="0 0 0"/>
-      <inertia ixx="0.0001" ixy="0" ixz="0" iyy="0.0001" iyz="0" izz="0.0001"/>
+      <mass value="0.1537"/>
+      <origin xyz="0.00000 -0.00000 -0.03428" rpy="0 0 0"/>
+      <inertia ixx="1.215946e-04" ixy="2.031805e-13" ixz="-3.218520e-13" iyy="1.215946e-04" iyz="3.146202e-10" izz="3.597206e-05"/>
     </inertial>
   </link>
