Commit message: feat: add D405 camera wrist mount to the robot collision model
The eye-in-hand D405 sits on a printed bracket whose pro630 ring (r=30mm) bolts to the
link6 flange between the arm and the suction cup. Add it everywhere planning sees the robot:
- URDF: new `camera_mount` link (STL mesh, visual + collision) fixed to link6
  (STL +Z -> flange axis, +Y -> link6 -Y toward the camera; ring centre at the flange).
- cuRobo (v1 source; planner regenerates v2 via port_v1_to_v2): camera_mount in
  collision_link_names + collision_spheres (ring + arm + D405 case) + self_collision_ignore
  (link4/5/6/suction_cup) + buffer. Verified: planner reloads, base + descent plans succeed
  with no spurious self-collisions, so the carried/angled-approach moves now avoid the mount.

Co-Authored-By: Claude Opus 4.8 <noreply@anthropic.com>

File: src/mycobot_description/urdf/mycobot_pro_630.urdf (robot description, URDF)
Before this commit: robot mycobot_pro_630, 11 links, 10 joints
Links:
- added link camera_mount, mass 0.05; collision mesh filename=package://mycobot_description/meshes/d405_case_ring_offset7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 scale=0.001 0.001 0.001; visual mesh filename=package://mycobot_description/meshes/d405_case_ring_offset7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 scale=0.001 0.001 0.001
- link base: mass 1.0 -> 3.4225
- link link1: mass 0.5 -> 0.5434
- link link2: mass 0.4 -> 1.8125
- link link3: mass 0.3 -> 2.2651
- link link4: mass 0.2 -> 0.3447
- link link5: mass 0.15 -> 0.4204
- link link6: mass 0.1 -> 0.0376
- link suction_cup: mass 0.05 -> 0.1537
Joints:
- added joint camera_mount_joint: type fixed, parent link6, child camera_mount, origin xyz=-0.003 -0.003 0 rpy=3.1416 1.5708 0
- joint tcp_joint: origin xyz=0 0 0.06 rpy=0 0 0 -> xyz=0 0 -0.145 rpy=3.1416 0 0

Commit message: Recalibrate suction-cup tcp 0.145 -> 0.135 m (cup shortened ~10mm)
A J2-shoulder-torque floor touch-test (pick_and_place/calib_z.py) on 2026-07-01 showed
the cup only first-touched the table when the model put the tip at z ~ -10mm, i.e. the
suction cup had taken a ~10mm compression set from repeated hard-press contact tests.
That made every touch/grasp land high and miss objects. tcp_joint origin -0.145 -> -0.135;
validated after a planner restart (cup now first-touches the table at model z ~ 0).

Co-Authored-By: Claude Opus 4.8 <noreply@anthropic.com>

File: src/mycobot_description/urdf/mycobot_pro_630.urdf (robot description, URDF)
Before this commit: robot mycobot_pro_630, 12 links, 11 joints
Joints:
- joint tcp_joint: origin xyz=0 0 -0.145 rpy=3.1416 0 0 -> xyz=0 0 -0.135 rpy=3.1416 0 0

Commit message: Pro 630 limits: URDF joint velocity 0.6283 rad/s (36 deg/s firmware ceiling), effort 186/50 Nm; cuRobo max_acceleration 10.47 rad/s^2
Co-Authored-By: Claude Fable 5.1 <noreply@anthropic.com>
Claude-Session: https://claude.ai/code/session_01GxmdNa4EPJY8gCWMzznLfT

File: src/mycobot_description/urdf/mycobot_pro_630.urdf (robot description, URDF)
Before this commit: robot mycobot_pro_630, 12 links, 11 joints
Joints:
- joint joint1: limit lower=-3.14159 upper=3.14159 effort=1000.0 velocity=1.5 -> lower=-3.14159 upper=3.14159 effort=186.0 velocity=0.6283
- joint joint2: limit lower=-3.14159 upper=3.14159 effort=1000.0 velocity=1.5 -> lower=-3.14159 upper=3.14159 effort=186.0 velocity=0.6283
- joint joint3: limit lower=-2.61 upper=2.618 effort=1000.0 velocity=1.5 -> lower=-2.61 upper=2.618 effort=186.0 velocity=0.6283
- joint joint4: limit lower=-2.9670 upper=2.9670 effort=1000.0 velocity=1.5 -> lower=-2.9670 upper=2.9670 effort=50.0 velocity=0.6283
- joint joint5: limit lower=-2.93 upper=2.9321 effort=1000.0 velocity=1.5 -> lower=-2.93 upper=2.9321 effort=50.0 velocity=0.6283
- joint joint6: limit lower=-3.03 upper=3.0368 effort=1000.0 velocity=1.5 -> lower=-3.03 upper=3.0368 effort=50.0 velocity=0.6283
